Commit message: week1_2

File: description/robot.urdf (robot description, URDF)
Before this commit: robot robot, 5 links, 4 joints
Links:
- added link laser_frame, mass 0.1; collision cylinder length=0.04 radius=0.05; visual cylinder length=0.04 radius=0.05
Joints:
- added joint laser_joint: type fixed, parent chassis, child laser_frame, origin xyz=0.1 0 0.175 rpy=0 0 0

File: description/robot.urdf.xacro (robot description, xacro)
@@ -2,3 +2,5 @@
 <robot xmlns:xacro="http://www.ros.org/wiki/xacro"  name="robot">
     <xacro:include filename="robot_core.xacro" />
+    <xacro:include filename="gazebo_control.xacro" />
+    <xacro:include filename="lidar.xacro" />
 </robot>
